File: pcbSmd/pcb.sch (KiCad schematic (older format))
At the start: 33 parts, among them J1 Conn_01x03_Male, J2 Conn_01x06_Male, P1 CONN_01X04, P2 CONN_01X04, Q1 2N7002, U1 TPS62160DGKT, U2 APX823-29 (-26 non disponible)

Commit message: je sais plus
Parts:
- C2: value 330pF -> 1.5nF
- D1, D2, D4, D6: symbol Diode:BAT60A -> pcb-rescue:BAT60A-Diode
- R1: value 10k -> 2.7k
- U2: symbol pcb-rescue:APX823-lib -> pcb-rescue:APX823-lib-pcb-rescue
Changed lines of the file:
@@
 EESchema Schematic File Version 4
-EELAYER 30 0
+LIBS:pcb-cache
+EELAYER 26 0
 EELAYER END
 $Descr A4 11693 8268
@@
 P 3650 2800
 F 0 "C2" H 3650 2900 50  0000 L CNN
-F 1 "330pF" H 3650 2700 50  0000 L CNN
+F 1 "1.5nF" H 3650 2700 50  0000 L CNN
 F 2 "Capacitor_SMD:C_0603_1608Metric_Pad1.08x0.95mm_HandSolder" H 3688 2650 50  0001 C CNN
 F 3 "" H 3650 2800 50  0000 C CNN
@@
 P 2750 2450
 F 0 "R1" H 2820 2496 50  0000 L CNN
-F 1 "10k" H 2820 2405 50  0000 L CNN
+F 1 "2.7k" H 2820 2405 50  0000 L CNN
 F 2 "Resistor_SMD:R_0603_1608Metric_Pad0.98x0.95mm_HandSolder" V 2680 2450 50  0001 C CNN
 F 3 "" H 2750 2450 50  0000 C CNN
@@
 	2600 1400 2800 1400
 $Comp
-L Diode:BAT60A D1
+L pcb-rescue:BAT60A-Diode D1
 U 1 1 60DF7455
 P 2800 1550
@@
 $EndComp
 $Comp
-L Diode:BAT60A D2
+L pcb-rescue:BAT60A-Diode D2
 U 1 1 60DF81BB
 P 3150 1400
@@
 	2300 4950 2300 5350
 $Comp
-L Diode:BAT60A D4
+L pcb-rescue:BAT60A-Diode D4
 U 1 1 60E31E82
 P 2450 5350
@@
 Connection ~ 2300 4550
 $Comp
-L pcb-rescue:APX823-lib U2
+L pcb-rescue:APX823-lib-pcb-rescue U2
 U 1 1 60EAFA97
 P 5600 3500
@@
 $EndComp
 $Comp
-L Diode:BAT60A D6
+L pcb-rescue:BAT60A-Diode D6
 U 1 1 60D5D5AB
 P 5150 3150
