File: pcbSmd/pcb.sync-conflict-20230220-230307-7RYDY7R.sch (KiCad schematic (older format))
At the start: 30 parts, among them J1 Conn_01x03_Male, J2 Conn_01x06_Male, P1 CONN_01X04, P2 CONN_01X04, Q1 2N7002, U1 TPS62160DGKT, U2 APX823-29 (-26 non disponible)

Commit message: je sais plus
Parts:
- added C?: 220uF 16V, Capacitor_THT:CP_Radial_D12.5mm_P5.00mm, symbol pcb-rescue:C-base-rescue
- added C?_missingOnBoard: 100nF, Capacitor_SMD:C_0603_1608Metric_Pad1.08x0.95mm_HandSolder, symbol pcb-rescue:C-base-rescue
- added R?_missingOnBoard: 100, Resistor_SMD:R_0603_1608Metric_Pad0.98x0.95mm_HandSolder, symbol pcb-rescue:R-base-rescue
- C2: value 330pF -> 1.5nF
- D1, D2, D4, D6: symbol Diode:BAT60A -> pcb-rescue:BAT60A-Diode
- D5: value BZT52C13S -> BZT52C13S remplacer par BZT52C14S
- R1: value 10k -> 4.7k
Connections:
- net +2V5: now also C?_missingOnBoard.1
- net GND: now also C?.2, C?_missingOnBoard.2
- net RST: now also R?_missingOnBoard.1; no longer U2.1 (~RESET)
- net VCC: now also C?.1
- new net: R?_missingOnBoard.2, U2.1 (~RESET)
Changed lines of the file:
@@
 EESchema Schematic File Version 4
-EELAYER 30 0
+LIBS:pcb-cache
+EELAYER 26 0
 EELAYER END
 $Descr A4 11693 8268
@@
 P 3650 2800
 F 0 "C2" H 3650 2900 50  0000 L CNN
-F 1 "330pF" H 3650 2700 50  0000 L CNN
+F 1 "1.5nF" H 3650 2700 50  0000 L CNN
 F 2 "Capacitor_SMD:C_0603_1608Metric_Pad1.08x0.95mm_HandSolder" H 3688 2650 50  0001 C CNN
 F 3 "" H 3650 2800 50  0000 C CNN
@@
 P 2750 2450
 F 0 "R1" H 2820 2496 50  0000 L CNN
-F 1 "10k" H 2820 2405 50  0000 L CNN
+F 1 "4.7k" H 2820 2405 50  0000 L CNN
 F 2 "Resistor_SMD:R_0603_1608Metric_Pad0.98x0.95mm_HandSolder" V 2680 2450 50  0001 C CNN
 F 3 "" H 2750 2450 50  0000 C CNN
@@
 	2600 1400 2800 1400
 $Comp
-L Diode:BAT60A D1
+L pcb-rescue:BAT60A-Diode D1
 U 1 1 60DF7455
 P 2800 1550
@@
 $EndComp
 $Comp
-L Diode:BAT60A D2
+L pcb-rescue:BAT60A-Diode D2
 U 1 1 60DF81BB
 P 3150 1400
@@
 	2300 4950 2300 5350
 $Comp
-L Diode:BAT60A D4
+L pcb-rescue:BAT60A-Diode D4
 U 1 1 60E31E82
 P 2450 5350
@@
 P 2300 4700
 F 0 "D5" V 2250 4550 50  0000 L CNN
-F 1 "BZT52C13S" V 2400 4250 50  0000 L CNN
+F 1 "BZT52C13S remplacer par BZT52C14S" V 2400 4250 50  0000 L CNN
 F 2 "Diode_SMD:D_SOD-323" H 2300 4525 50  0001 C CNN
 F 3 "https://diotec.com/tl_files/diotec/files/pdf/datasheets/bzt52b2v4.pdf" H 2300 4700 50  0001 C CNN
@@
 	1    0    0    -1
 $EndComp
-Text Label 6000 3500 0    50   ~ 0
+Text Label 6300 3500 0    50   ~ 0
 RST
 $Comp
@@
 $EndComp
 $Comp
-L Diode:BAT60A D6
+L pcb-rescue:BAT60A-Diode D6
 U 1 1 60D5D5AB
 P 5150 3150
@@
 	0    1    1    0
 $EndComp
+$Comp
+L pcb-rescue:C-base-rescue C?_missingOnBoard
+U 1 1 61216729
+P 5250 4750
+F 0 "C?_missingOnBoard" H 5275 4850 50  0000 L CNN
+F 1 "100nF" H 5275 4650 50  0000 L CNN
+F 2 "Capacitor_SMD:C_0603_1608Metric_Pad1.08x0.95mm_HandSolder" H 5288 4600 50  0001 C CNN
+F 3 "" H 5250 4750 50  0000 C CNN
+	1    5250 4750
+	1    0    0    -1
+$EndComp
+Wire Wire Line
+	4900 4550 5250 4550
+Wire Wire Line
+	5250 4550 5250 4600
+$Comp
+L power:GND #PWR?
+U 1 1 61217F20
+P 5250 4900
+F 0 "#PWR?" H 5250 4650 50  0001 C CNN
+F 1 "GND" H 5250 4750 50  0000 C CNN
+F 2 "" H 5250 4900 50  0000 C CNN
+F 3 "" H 5250 4900 50  0000 C CNN
+	1    5250 4900
+	1    0    0    -1
+$EndComp
+$Comp
+L pcb-rescue:R-base-rescue R?_missingOnBoard
+U 1 1 6121E376
+P 6150 3500
+F 0 "R?_missingOnBoard" V 6250 3650 50  0000 C CNN
+F 1 "100" V 6150 3500 50  0000 C CNN
+F 2 "Resistor_SMD:R_0603_1608Metric_Pad0.98x0.95mm_HandSolder" V 6080 3500 50  0001 C CNN
+F 3 "" H 6150 3500 50  0000 C CNN
+	1    6150 3500
+	0    1    1    0
+$EndComp
+$Comp
+L pcb-rescue:C-base-rescue C?
+U 1 1 61249EA2
+P 5250 1550
+F 0 "C?" H 5365 1596 50  0000 L CNN
+F 1 "220uF 16V" H 5250 1450 50  0000 L CNN
+F 2 "Capacitor_THT:CP_Radial_D12.5mm_P5.00mm" H 5288 1400 50  0001 C CNN
+F 3 "" H 5250 1550 50  0000 C CNN
+F 4 "13x25mm" H 5500 1350 50  0000 C CNN "Field4"
+	1    5250 1550
+	1    0    0    -1
+$EndComp
+Wire Wire Line
+	4600 1400 5250 1400
+$Comp
+L power:GND #PWR?
+U 1 1 6124BF93
+P 5250 1700
+F 0 "#PWR?" H 5250 1450 50  0001 C CNN
+F 1 "GND" H 5255 1527 50  0000 C CNN
+F 2 "" H 5250 1700 50  0001 C CNN
+F 3 "" H 5250 1700 50  0001 C CNN
+	1    5250 1700
+	1    0    0    -1
+$EndComp
 $EndSCHEMATC
