File: pcbSmd/pcb.kicad_sch (KiCad schematic)
At the start: 33 parts, among them J1 Conn_01x03_Male, J2 Conn_01x06_Male, P1 CONN_01X04, P2 CONN_01X04, Q1 2N7002, U1 TPS62160DGKT, U2 APX823-29 (-26 non disponible)

Commit message: Quelque correction de valeur.
Parts:
- C2: value 1.5nF -> 10nF
- R3: value 10k -> 100k
Changed lines of the file:
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@@
       (effects (font (size 1.27 1.27)) (justify left))
     )
-    (property "Value" "1.5nF" (id 1) (at 92.71 73.66 0)
+    (property "Value" "10nF" (id 1) (at 92.71 73.66 0)
       (effects (font (size 1.27 1.27)) (justify left))
     )
@@
       (effects (font (size 1.27 1.27)) (justify left))
     )
-    (property "Value" "10k" (id 1) (at 57.658 43.053 0)
+    (property "Value" "100k" (id 1) (at 57.658 43.053 0)
       (effects (font (size 1.27 1.27)) (justify left))
     )
@@
     )
     (path "/00000000-0000-0000-0000-00005fdfe767"
-      (reference "C2") (unit 1) (value "1.5nF") (footprint "Capacitor_SMD:C_0603_1608Metric_Pad1.08x0.95mm_HandSolder")
+      (reference "C2") (unit 1) (value "10nF") (footprint "Capacitor_SMD:C_0603_1608Metric_Pad1.08x0.95mm_HandSolder")
     )
     (path "/00000000-0000-0000-0000-00005fdebce2"
@@
     )
     (path "/00000000-0000-0000-0000-00005fe1b5a7"
-      (reference "R3") (unit 1) (value "10k") (footprint "Resistor_SMD:R_0603_1608Metric_Pad0.98x0.95mm_HandSolder")
+      (reference "R3") (unit 1) (value "100k") (footprint "Resistor_SMD:R_0603_1608Metric_Pad0.98x0.95mm_HandSolder")
     )
     (path "/00000000-0000-0000-0000-000060d6fe11"
